Commit message: Humanoid Robot v1.7.0: Introduce pelvis based humanoid skeleton

File: src/humanoid_description/backup/humanoid_v1.5_before_pelvis.xacro (robot description, xacro)
@@ -1,5 +1,5 @@
 <?xml version="1.0"?>
 <robot xmlns:xacro="http://www.ros.org/wiki/xacro"
-       name="humanoid_v1_7">
+       name="humanoid_v1_5">
   <!-- ================= -->
   <!-- Include Modules -->
@@ -7,64 +7,55 @@
   <xacro:include
     filename="$(find humanoid_description)/urdf/modules/legs.xacro"/>
-  <xacro:include
-    filename="$(find humanoid_description)/urdf/modules/pelvis.xacro"/>
   <!-- ================= -->
-  <!-- Robot Root -->
+  <!-- Base -->
   <!-- ================= -->
   <link name="base_link">
+    <visual>
+      <geometry>
+        <box size="0.4 0.25 0.5"/>
+      </geometry>
+      <origin xyz="0 0 0.25"/>
+      <material name="blue">
+        <color rgba="0 0 1 1"/>
+      </material>
+    </visual>
   </link>
   <!-- ================= -->
-  <!-- Pelvis -->
-  <!-- ================= -->
-  <xacro:pelvis/>
-  <!-- ================= -->
-  <!-- Base To Pelvis -->
-  <!-- ================= -->
-  <joint name="base_to_pelvis"
-         type="fixed">
-    <parent link="base_link"/>
-    <child link="pelvis_link"/>
-    <origin
-      xyz="0 0 0.85"/>
-  </joint>
-  <!-- ================= -->
-  <!-- Legs -->
+  <!-- Left Leg -->
   <!-- ================= -->
   <xacro:leg
     prefix="left"/>
+  <!-- ================= -->
+  <!-- Right Leg -->
+  <!-- ================= -->
   <xacro:leg
     prefix="right"/>
   <!-- ================= -->
-  <!-- Left Hip -->
+  <!-- Hip Joints -->
   <!-- ================= -->
   <joint name="left_hip_joint"
          type="revolute">
-    <parent link="pelvis_link"/>
+    <parent link="base_link"/>
     <child link="left_thigh"/>
     <origin
       xyz="0 0.15 0"/>
-    <axis
-      xyz="1 0 0"/>
+    <axis xyz="1 0 0"/>
     <limit
       lower="-1.57"
       upper="1.57"
-      effort="20"
+      effort="10"
       velocity="1"/>
   </joint>
-  <!-- ================= -->
-  <!-- Right Hip -->
-  <!-- ================= -->
   <joint name="right_hip_joint"
          type="revolute">
-    <parent link="pelvis_link"/>
+    <parent link="base_link"/>
     <child link="right_thigh"/>
     <origin
       xyz="0 -0.15 0"/>
-    <axis
-      xyz="1 0 0"/>
+    <axis xyz="1 0 0"/>
     <limit
       lower="-1.57"
       upper="1.57"
-      effort="20"
+      effort="10"
       velocity="1"/>
   </joint>

File: src/humanoid_description/backup/legs_v1.5.3_before_inertial.xacro (robot description, xacro)
@@ -1,5 +1,7 @@
 <?xml version="1.0"?>
 <robot xmlns:xacro="http://www.ros.org/wiki/xacro">
+  <!-- ===================== -->
   <!-- Materials -->
+  <!-- ===================== -->
   <material name="gray">
     <color rgba="0.5 0.5 0.5 1"/>
@@ -11,10 +13,10 @@
     <color rgba="0.1 0.1 0.1 1"/>
   </material>
-  <!-- Leg Macro -->
+  <!-- ===================== -->
+  <!-- Leg Link Macro -->
+  <!-- ===================== -->
   <xacro:macro name="leg"
-               params="prefix">
-    <!-- ================= -->
+               params="prefix ">
     <!-- thigh -->
-    <!-- ================= -->
     <link name="${prefix}_thigh">
       <visual>
@@ -28,29 +30,6 @@
         <material name="gray"/>
       </visual>
-      <collision>
-        <geometry>
-          <cylinder
-            radius="0.06"
-            length="0.35"/>
-        </geometry>
-        <origin
-          xyz="0 0 -0.175"/>
-      </collision>
-      <inertial>
-        <mass value="1.0"/>
-        <origin
-          xyz="0 0 -0.175"/>
-        <inertia
-          ixx="0.01"
-          ixy="0"
-          ixz="0"
-          iyy="0.01"
-          iyz="0"
-          izz="0.002"/>
-      </inertial>
     </link>
-    <!-- ================= -->
     <!-- shin -->
-    <!-- ================= -->
     <link name="${prefix}_shin">
       <visual>
@@ -64,29 +43,6 @@
         <material name="dark_gray"/>
       </visual>
-      <collision>
-        <geometry>
-          <cylinder
-            radius="0.05"
-            length="0.35"/>
-        </geometry>
-        <origin
-          xyz="0 0 -0.175"/>
-      </collision>
-      <inertial>
-        <mass value="0.7"/>
-        <origin
-          xyz="0 0 -0.175"/>
-        <inertia
-          ixx="0.006"
-          ixy="0"
-          ixz="0"
-          iyy="0.006"
-          iyz="0"
-          izz="0.001"/>
-      </inertial>
     </link>
-    <!-- ================= -->
     <!-- foot -->
-    <!-- ================= -->
     <link name="${prefix}_foot">
       <visual>
@@ -98,23 +54,4 @@
         <material name="black"/>
       </visual>
-      <collision>
-        <geometry>
-          <box size="0.25 0.15 0.08"/>
-        </geometry>
-        <origin
-          xyz="0.08 0 -0.04"/>
-      </collision>
-      <inertial>
-        <mass value="0.3"/>
-        <origin
-          xyz="0.08 0 -0.04"/>
-        <inertia
-          ixx="0.001"
-          ixy="0"
-          ixz="0"
-          iyy="0.002"
-          iyz="0"
-          izz="0.002"/>
-      </inertial>
     </link>
     <!-- knee -->
