Commit message: Humanoid Robot v1.9: Complete humanoid body assembly with arms head and joint GUI

File: src/humanoid_description/backup/humanoid_v1.7_before_v1.9.xacro (robot description, xacro)
@@ -1,5 +1,5 @@
 <?xml version="1.0"?>
 <robot xmlns:xacro="http://www.ros.org/wiki/xacro"
-       name="humanoid_v1_9">
+       name="humanoid_v1_7">
   <!-- ================= -->
   <!-- Include Modules -->
@@ -9,18 +9,16 @@
   <xacro:include
     filename="$(find humanoid_description)/urdf/modules/pelvis.xacro"/>
-  <xacro:include
-    filename="$(find humanoid_description)/urdf/modules/torso.xacro"/>
-  <xacro:include
-    filename="$(find humanoid_description)/urdf/modules/arms.xacro"/>
-  <xacro:include
-    filename="$(find humanoid_description)/urdf/modules/head.xacro"/>
   <!-- ================= -->
-  <!-- Root Link -->
+  <!-- Robot Root -->
   <!-- ================= -->
-  <link name="base_link"/>
+  <link name="base_link">
+  </link>
   <!-- ================= -->
   <!-- Pelvis -->
   <!-- ================= -->
   <xacro:pelvis/>
+  <!-- ================= -->
+  <!-- Base To Pelvis -->
+  <!-- ================= -->
   <joint name="base_to_pelvis"
          type="fixed">
@@ -31,19 +29,13 @@
   </joint>
   <!-- ================= -->
-  <!-- Torso -->
-  <!-- ================= -->
-  <xacro:torso/>
-  <joint name="pelvis_to_torso"
-         type="fixed">
-    <parent link="pelvis_link"/>
-    <child link="torso_link"/>
-    <origin
-      xyz="0 0 0.35"/>
-  </joint>
-  <!-- ================= -->
   <!-- Legs -->
   <!-- ================= -->
-  <xacro:leg prefix="left"/>
-  <xacro:leg prefix="right"/>
+  <xacro:leg
+    prefix="left"/>
+  <xacro:leg
+    prefix="right"/>
+  <!-- ================= -->
+  <!-- Left Hip -->
+  <!-- ================= -->
   <joint name="left_hip_joint"
          type="revolute">
@@ -52,18 +44,6 @@
     <origin
       xyz="0 0.15 0"/>
-    <axis xyz="1 0 0"/>
-    <limit
-      lower="-1.57"
-      upper="1.57"
-      effort="20"
-      velocity="1"/>
-  </joint>
-  <joint name="right_hip_joint"
-         type="revolute">
-    <parent link="pelvis_link"/>
-    <child link="right_thigh"/>
-    <origin
-      xyz="0 -0.15 0"/>
-    <axis xyz="1 0 0"/>
+    <axis
+      xyz="1 0 0"/>
     <limit
       lower="-1.57"
@@ -73,15 +53,19 @@
   </joint>
   <!-- ================= -->
-  <!-- Arms -->
+  <!-- Right Hip -->
   <!-- ================= -->
-  <xacro:arm
-    prefix="left"
-    side="0.25"/>
-  <xacro:arm
-    prefix="right"
-    side="-0.25"/>
-  <!-- ================= -->
-  <!-- Head -->
-  <!-- ================= -->
-  <xacro:head/>
+  <joint name="right_hip_joint"
+         type="revolute">
+    <parent link="pelvis_link"/>
+    <child link="right_thigh"/>
+    <origin
+      xyz="0 -0.15 0"/>
+    <axis
+      xyz="1 0 0"/>
+    <limit
+      lower="-1.57"
+      upper="1.57"
+      effort="20"
+      velocity="1"/>
+  </joint>
 </robot>

File: src/humanoid_description/backup/torso_v1.9_before_fix.xacro (robot description, xacro)
@@ -34,4 +34,11 @@
       </inertial>
     </link>
+    <joint name="torso_joint"
+           type="fixed">
+      <parent link="base_link"/>
+      <child link="torso_link"/>
+      <origin
+        xyz="0 0 0.55"/>
+    </joint>
   </xacro:macro>
 </robot>
