Commit message: Humanoid Robot v2.0.0: Add articulated arms with shoulder joints

File: src/humanoid_description/backup/arms_v2.0_before_dynamics.xacro (robot description, xacro)
@@ -1,26 +1,24 @@
 <?xml version="1.0"?>
 <robot xmlns:xacro="http://www.ros.org/wiki/xacro">
-  <!-- ===================== -->
+  <!-- ================= -->
   <!-- Materials -->
-  <!-- ===================== -->
+  <!-- ================= -->
   <material name="arm_gray">
-    <color rgba="0.65 0.65 0.65 1"/>
+    <color rgba="0.45 0.45 0.45 1"/>
   </material>
   <material name="hand_black">
     <color rgba="0.1 0.1 0.1 1"/>
   </material>
-  <!-- ===================== -->
+  <!-- ================= -->
   <!-- Arm Macro -->
-  <!-- ===================== -->
+  <!-- ================= -->
   <xacro:macro name="arm"
                params="prefix side">
-    <!-- ================= -->
     <!-- Upper Arm -->
-    <!-- ================= -->
     <link name="${prefix}_upper_arm">
       <visual>
         <geometry>
           <cylinder
-            radius="0.045"
+            radius="0.05"
             length="0.30"/>
         </geometry>
@@ -32,5 +30,39 @@
         <geometry>
           <cylinder
-            radius="0.045"
+            radius="0.05"
+            length="0.30"/>
+        </geometry>
+        <origin
+          xyz="0 0 -0.15"/>
+      </collision>
+      <inertial>
+        <mass value="1.0"/>
+        <origin
+          xyz="0 0 -0.15"/>
+        <inertia
+          ixx="0.01"
+          ixy="0"
+          ixz="0"
+          iyy="0.01"
+          iyz="0"
+          izz="0.005"/>
+      </inertial>
+    </link>
+    <!-- Forearm -->
+    <link name="${prefix}_forearm">
+      <visual>
+        <geometry>
+          <cylinder
+            radius="0.04"
+            length="0.30"/>
+        </geometry>
+        <origin
+          xyz="0 0 -0.15"/>
+        <material name="arm_gray"/>
+      </visual>
+      <collision>
+        <geometry>
+          <cylinder
+            radius="0.04"
             length="0.30"/>
         </geometry>
@@ -43,39 +75,33 @@
           xyz="0 0 -0.15"/>
         <inertia
-          ixx="0.006"
+          ixx="0.008"
           ixy="0"
           ixz="0"
-          iyy="0.006"
+          iyy="0.008"
           iyz="0"
-          izz="0.001"/>
+          izz="0.004"/>
       </inertial>
     </link>
-    <!-- ================= -->
-    <!-- Forearm -->
-    <!-- ================= -->
-    <link name="${prefix}_forearm">
+    <!-- Hand -->
+    <link name="${prefix}_hand">
       <visual>
         <geometry>
-          <cylinder
-            radius="0.035"
-            length="0.25"/>
+          <box size="0.12 0.08 0.18"/>
         </geometry>
         <origin
-          xyz="0 0 -0.125"/>
-        <material name="arm_gray"/>
+          xyz="0 0 -0.09"/>
+        <material name="hand_black"/>
       </visual>
       <collision>
         <geometry>
-          <cylinder
-            radius="0.035"
-            length="0.25"/>
+          <box size="0.12 0.08 0.18"/>
         </geometry>
         <origin
-          xyz="0 0 -0.125"/>
+          xyz="0 0 -0.09"/>
       </collision>
       <inertial>
-        <mass value="0.5"/>
+        <mass value="0.3"/>
         <origin
-          xyz="0 0 -0.125"/>
+          xyz="0 0 -0.09"/>
         <inertia
           ixx="0.003"
@@ -84,42 +110,8 @@
           iyy="0.003"
           iyz="0"
-          izz="0.0008"/>
+          izz="0.002"/>
       </inertial>
     </link>
-    <!-- ================= -->
-    <!-- Hand -->
-    <!-- ================= -->
-    <link name="${prefix}_hand">
-      <visual>
-        <geometry>
-          <box size="0.12 0.08 0.05"/>
-        </geometry>
-        <origin
-          xyz="0 -0.02 -0.025"/>
-        <material name="hand_black"/>
-      </visual>
-      <collision>
-        <geometry>
-          <box size="0.12 0.08 0.05"/>
-        </geometry>
-        <origin
-          xyz="0 -0.02 -0.025"/>
-      </collision>
-      <inertial>
-        <mass value="0.2"/>
-        <origin
-          xyz="0 -0.02 -0.025"/>
-        <inertia
-          ixx="0.0005"
-          ixy="0"
-          ixz="0"
-          iyy="0.0005"
-          iyz="0"
-          izz="0.0005"/>
-      </inertial>
-    </link>
-    <!-- ================= -->
     <!-- Shoulder Joint -->
-    <!-- ================= -->
     <joint name="${prefix}_shoulder_joint"
            type="revolute">
@@ -128,14 +120,13 @@
       <origin
         xyz="0 ${side} 0.15"/>
-      <axis xyz="1 0 0"/>
+      <axis
+        xyz="1 0 0"/>
       <limit
         lower="-1.57"
         upper="1.57"
-        effort="30"
-        velocity="2"/>
+        effort="20"
+        velocity="1"/>
     </joint>
-    <!-- ================= -->
     <!-- Elbow Joint -->
-    <!-- ================= -->
     <joint name="${prefix}_elbow_joint"
            type="revolute">
@@ -144,14 +135,13 @@
       <origin
         xyz="0 0 -0.30"/>
-      <axis xyz="1 0 0"/>
+      <axis
+        xyz="1 0 0"/>
       <limit
-        lower="-2.0"
-        upper="0"
-        effort="20"
-        velocity="2"/>
+        lower="0"
+        upper="2.5"
+        effort="15"
+        velocity="1"/>
     </joint>
-    <!-- ================= -->
-    <!-- Wrist Joint -->
-    <!-- ================= -->
+    <!-- Wrist -->
     <joint name="${prefix}_wrist_joint"
            type="fixed">
@@ -159,5 +149,5 @@
       <child link="${prefix}_hand"/>
       <origin
-        xyz="0 0 -0.25"/>
+        xyz="0 0 -0.30"/>
     </joint>
   </xacro:macro>

File: src/humanoid_description/backup/arms_v2.0_before_shoulder_joint_fix.xacro (robot description, xacro)
@@ -19,4 +19,17 @@
     <!-- ================= -->
     <link name="${prefix}_upper_arm">
+<joint name="${prefix}_shoulder_joint"
+       type="revolute">
+  <parent link="torso_link"/>
+  <child link="${prefix}_upper_arm"/>
+  <origin
+    xyz="0 ${side} 0.15"/>
+  <axis xyz="1 0 0"/>
+  <limit
+    lower="-1.57"
+    upper="1.57"
+    effort="30"
+    velocity="2"/>
+</joint>
       <visual>
         <geometry>
@@ -120,24 +133,8 @@
     </link>
     <!-- ================= -->
-    <!-- Shoulder Joint -->
-    <!-- ================= -->
-    <joint name="${prefix}_shoulder_joint"
-           type="revolute">
-      <parent link="torso_link"/>
-      <child link="${prefix}_upper_arm"/>
-      <origin
-        xyz="0 ${side} 0.15"/>
-      <axis xyz="1 0 0"/>
-      <limit
-        lower="-1.57"
-        upper="1.57"
-        effort="30"
-        velocity="2"/>
-    </joint>
-    <!-- ================= -->
     <!-- Elbow Joint -->
     <!-- ================= -->
     <joint name="${prefix}_elbow_joint"
-           type="revolute">
+            type="revolute">
       <parent link="${prefix}_upper_arm"/>
       <child link="${prefix}_forearm"/>
@@ -148,5 +145,5 @@
         lower="-2.0"
         upper="0"
-        effort="20"
+        effort="30"
         velocity="2"/>
     </joint>
@@ -155,5 +152,5 @@
     <!-- ================= -->
     <joint name="${prefix}_wrist_joint"
-           type="fixed">
+            type="fixed">
       <parent link="${prefix}_forearm"/>
       <child link="${prefix}_hand"/>

File: src/humanoid_description/backup/arms_v2.0_before_side_fix.xacro (robot description, xacro)
@@ -14,5 +14,5 @@
   <!-- ===================== -->
   <xacro:macro name="arm"
-               params="prefix side">
+               params="prefix">
     <!-- ================= -->
     <!-- Upper Arm -->
@@ -120,24 +120,8 @@
     </link>
     <!-- ================= -->
-    <!-- Shoulder Joint -->
-    <!-- ================= -->
-    <joint name="${prefix}_shoulder_joint"
-           type="revolute">
-      <parent link="torso_link"/>
-      <child link="${prefix}_upper_arm"/>
-      <origin
-        xyz="0 ${side} 0.15"/>
-      <axis xyz="1 0 0"/>
-      <limit
-        lower="-1.57"
-        upper="1.57"
-        effort="30"
-        velocity="2"/>
-    </joint>
-    <!-- ================= -->
     <!-- Elbow Joint -->
     <!-- ================= -->
     <joint name="${prefix}_elbow_joint"
-           type="revolute">
+            type="revolute">
       <parent link="${prefix}_upper_arm"/>
       <child link="${prefix}_forearm"/>
@@ -148,5 +132,5 @@
         lower="-2.0"
         upper="0"
-        effort="20"
+        effort="30"
         velocity="2"/>
     </joint>
@@ -155,5 +139,5 @@
     <!-- ================= -->
     <joint name="${prefix}_wrist_joint"
-           type="fixed">
+            type="fixed">
       <parent link="${prefix}_forearm"/>
       <child link="${prefix}_hand"/>

File: src/humanoid_description/backup/legs_v2.0_before_dynamics.xacro (robot description, xacro)
@@ -1,20 +1,19 @@
 <?xml version="1.0"?>
 <robot xmlns:xacro="http://www.ros.org/wiki/xacro">
-  <!-- ===================== -->
   <!-- Materials -->
-  <!-- ===================== -->
-  <material name="leg_gray">
-    <color rgba="0.55 0.55 0.55 1"/>
+  <material name="gray">
+    <color rgba="0.5 0.5 0.5 1"/>
   </material>
-  <material name="foot_black">
+  <material name="dark_gray">
+    <color rgba="0.3 0.3 0.3 1"/>
+  </material>
+  <material name="black">
     <color rgba="0.1 0.1 0.1 1"/>
   </material>
-  <!-- ===================== -->
   <!-- Leg Macro -->
-  <!-- ===================== -->
   <xacro:macro name="leg"
                params="prefix">
     <!-- ================= -->
-    <!-- Thigh -->
+    <!-- thigh -->
     <!-- ================= -->
     <link name="${prefix}_thigh">
@@ -22,51 +21,15 @@
         <geometry>
           <cylinder
-            radius="0.065"
+            radius="0.06"
             length="0.35"/>
         </geometry>
         <origin
           xyz="0 0 -0.175"/>
-        <material name="leg_gray"/>
+        <material name="gray"/>
       </visual>
       <collision>
         <geometry>
           <cylinder
-            radius="0.065"
-            length="0.35"/>
-        </geometry>
-        <origin
-          xyz="0 0 -0.175"/>
-      </collision>
-      <inertial>
-        <mass value="1.5"/>
-        <origin
-          xyz="0 0 -0.175"/>
-        <inertia
-          ixx="0.015"
-          ixy="0"
-          ixz="0"
-          iyy="0.015"
-          iyz="0"
-          izz="0.003"/>
-      </inertial>
-    </link>
-    <!-- ================= -->
-    <!-- Shin -->
-    <!-- ================= -->
-    <link name="${prefix}_shin">
-      <visual>
-        <geometry>
-          <cylinder
-            radius="0.055"
-            length="0.35"/>
-        </geometry>
-        <origin
-          xyz="0 0 -0.175"/>
-        <material name="leg_gray"/>
-      </visual>
-      <collision>
-        <geometry>
-          <cylinder
-            radius="0.055"
+            radius="0.06"
             length="0.35"/>
         </geometry>
@@ -88,18 +51,54 @@
     </link>
     <!-- ================= -->
-    <!-- Foot -->
+    <!-- shin -->
+    <!-- ================= -->
+    <link name="${prefix}_shin">
+      <visual>
+        <geometry>
+          <cylinder
+            radius="0.05"
+            length="0.35"/>
+        </geometry>
+        <origin
+          xyz="0 0 -0.175"/>
+        <material name="dark_gray"/>
+      </visual>
+      <collision>
+        <geometry>
+          <cylinder
+            radius="0.05"
+            length="0.35"/>
+        </geometry>
+        <origin
+          xyz="0 0 -0.175"/>
+      </collision>
+      <inertial>
+        <mass value="0.7"/>
+        <origin
+          xyz="0 0 -0.175"/>
+        <inertia
+          ixx="0.006"
+          ixy="0"
+          ixz="0"
+          iyy="0.006"
+          iyz="0"
+          izz="0.001"/>
+      </inertial>
+    </link>
+    <!-- ================= -->
+    <!-- foot -->
     <!-- ================= -->
     <link name="${prefix}_foot">
       <visual>
         <geometry>
-          <box size="0.25 0.14 0.08"/>
+          <box size="0.25 0.15 0.08"/>
         </geometry>
         <origin
           xyz="0.08 0 -0.04"/>
-        <material name="foot_black"/>
+        <material name="black"/>
       </visual>
       <collision>
         <geometry>
-          <box size="0.25 0.14 0.08"/>
+          <box size="0.25 0.15 0.08"/>
         </geometry>
         <origin
@@ -107,21 +106,19 @@
       </collision>
       <inertial>
-        <mass value="0.5"/>
+        <mass value="0.3"/>
         <origin
           xyz="0.08 0 -0.04"/>
         <inertia
-          ixx="0.002"
+          ixx="0.001"
           ixy="0"
           ixz="0"
-          iyy="0.004"
+          iyy="0.002"
           iyz="0"
-          izz="0.005"/>
+          izz="0.002"/>
       </inertial>
     </link>
-    <!-- ================= -->
-    <!-- Knee Joint -->
-    <!-- ================= -->
+    <!-- knee -->
     <joint name="${prefix}_knee_joint"
-            type="revolute">
+           type="revolute">
       <parent link="${prefix}_thigh"/>
       <child link="${prefix}_shin"/>
@@ -132,12 +129,10 @@
         lower="0"
         upper="2.5"
-        effort="50"
-        velocity="2"/>
+        effort="10"
+        velocity="1"/>
     </joint>
-    <!-- ================= -->
-    <!-- Ankle Joint -->
-    <!-- ================= -->
+    <!-- ankle -->
     <joint name="${prefix}_ankle_joint"
-            type="fixed">
+           type="fixed">
       <parent link="${prefix}_shin"/>
       <child link="${prefix}_foot"/>
