Commit message: Humanoid Robot v2.5.0: Clean modular humanoid architecture

File: src/humanoid_description/backup/head_v2.5_before_clean.xacro (robot description, xacro)
@@ -7,6 +7,6 @@
     <color rgba="0.65 0.65 0.65 1"/>
   </material>
-  <material name="neck_dark">
-    <color rgba="0.25 0.25 0.25 1"/>
+  <material name="sensor_black">
+    <color rgba="0.05 0.05 0.05 1"/>
   </material>
   <!-- ================= -->
@@ -19,24 +19,24 @@
         <geometry>
           <cylinder
-            radius="0.06"
-            length="0.20"/>
+            radius="0.08"
+            length="0.15"/>
         </geometry>
         <origin
-          xyz="0 0 0"/>
-        <material name="neck_dark"/>
+          xyz="0 0 -0.075"/>
+        <material name="head_gray"/>
       </visual>
       <collision>
         <geometry>
           <cylinder
-            radius="0.06"
-            length="0.20"/>
+            radius="0.08"
+            length="0.15"/>
         </geometry>
         <origin
-          xyz="0 0 0"/>
+          xyz="0 0 -0.075"/>
       </collision>
       <inertial>
         <mass value="0.5"/>
         <origin
-          xyz="0 0 0"/>
+          xyz="0 0 -0.075"/>
         <inertia
           ixx="0.002"
@@ -45,5 +45,5 @@
           iyy="0.002"
           iyz="0"
-          izz="0.002"/>
+          izz="0.001"/>
       </inertial>
     </link>
@@ -52,5 +52,6 @@
       <visual>
         <geometry>
-          <sphere radius="0.18"/>
+          <sphere
+            radius="0.16"/>
         </geometry>
         <origin
@@ -60,5 +61,6 @@
       <collision>
         <geometry>
-          <sphere radius="0.18"/>
+          <sphere
+            radius="0.16"/>
         </geometry>
         <origin
@@ -70,12 +72,35 @@
           xyz="0 0 0"/>
         <inertia
-          ixx="0.005"
+          ixx="0.01"
           ixy="0"
           ixz="0"
-          iyy="0.005"
+          iyy="0.01"
           iyz="0"
-          izz="0.005"/>
+          izz="0.01"/>
       </inertial>
     </link>
+    <!-- Neck Joint -->
+    <joint name="neck_joint"
+           type="revolute">
+      <parent link="torso_link"/>
+      <child link="neck_link"/>
+      <origin
+        xyz="0 0 0.35"/>
+      <axis
+        xyz="0 1 0"/>
+      <limit
+        lower="-1.0"
+        upper="1.0"
+        effort="10"
+        velocity="1"/>
+    </joint>
+    <!-- Head Joint -->
+    <joint name="head_joint"
+           type="fixed">
+      <parent link="neck_link"/>
+      <child link="head_link"/>
+      <origin
+        xyz="0 0 0.15"/>
+    </joint>
   </xacro:macro>
 </robot>

File: src/humanoid_description/backup/pelvis_v2.5_before_clean.xacro (robot description, xacro)
@@ -1,19 +1,9 @@
 <?xml version="1.0"?>
 <robot xmlns:xacro="http://www.ros.org/wiki/xacro">
-  <!-- ===================== -->
-  <!-- Materials -->
-  <!-- ===================== -->
   <material name="pelvis_blue">
     <color rgba="0 0.3 1 1"/>
   </material>
-  <!-- ===================== -->
-  <!-- Pelvis Macro -->
-  <!-- ===================== -->
   <xacro:macro name="pelvis">
-    <!-- ================= -->
-    <!-- Pelvis Link -->
-    <!-- ================= -->
     <link name="pelvis_link">
-      <!-- Visual -->
       <visual>
         <geometry>
@@ -24,5 +14,4 @@
         <material name="pelvis_blue"/>
       </visual>
-      <!-- Collision -->
       <collision>
         <geometry>
@@ -32,5 +21,4 @@
           xyz="0 0 0"/>
       </collision>
-      <!-- Inertial -->
       <inertial>
         <mass value="2.5"/>
@@ -38,10 +26,10 @@
           xyz="0 0 0"/>
         <inertia
-          ixx="0.025"
+          ixx="0.02"
           ixy="0"
           ixz="0"
-          iyy="0.020"
+          iyy="0.02"
           iyz="0"
-          izz="0.015"/>
+          izz="0.01"/>
       </inertial>
     </link>

File: src/humanoid_description/backup/torso_v2.5_before_inertial_upgrade.xacro (robot description, xacro)
@@ -1,22 +1,12 @@
 <?xml version="1.0"?>
 <robot xmlns:xacro="http://www.ros.org/wiki/xacro">
-  <!-- ===================== -->
-  <!-- Materials -->
-  <!-- ===================== -->
   <material name="torso_blue">
-    <color rgba="0 0.3 1 1"/>
+    <color rgba="0 0 0.8 1"/>
   </material>
-  <!-- ===================== -->
-  <!-- Torso Macro -->
-  <!-- ===================== -->
   <xacro:macro name="torso">
-    <!-- ================= -->
-    <!-- Torso Link -->
-    <!-- ================= -->
     <link name="torso_link">
-      <!-- Visual -->
       <visual>
         <geometry>
-          <box size="0.45 0.30 0.55"/>
+          <box size="0.45 0.3 0.55"/>
         </geometry>
         <origin
@@ -24,13 +14,11 @@
         <material name="torso_blue"/>
       </visual>
-      <!-- Collision -->
       <collision>
         <geometry>
-          <box size="0.45 0.30 0.55"/>
+          <box size="0.45 0.3 0.55"/>
         </geometry>
         <origin
           xyz="0 0 0"/>
       </collision>
-      <!-- Inertial -->
       <inertial>
         <mass value="5.0"/>
@@ -38,10 +26,10 @@
           xyz="0 0 0"/>
         <inertia
-          ixx="0.12"
+          ixx="0.05"
           ixy="0"
           ixz="0"
-          iyy="0.10"
+          iyy="0.05"
           iyz="0"
-          izz="0.08"/>
+          izz="0.03"/>
       </inertial>
     </link>

File: src/humanoid_description/backup/torso_v2.5_duplicate_fix.xacro (robot description, xacro)
@@ -4,28 +4,28 @@
   <!-- Materials -->
   <!-- ===================== -->
-  <material name="pelvis_blue">
+  <material name="torso_blue">
     <color rgba="0 0.3 1 1"/>
   </material>
   <!-- ===================== -->
-  <!-- Pelvis Macro -->
+  <!-- Torso Macro -->
   <!-- ===================== -->
-  <xacro:macro name="pelvis">
+  <xacro:macro name="torso">
     <!-- ================= -->
-    <!-- Pelvis Link -->
+    <!-- Torso Link -->
     <!-- ================= -->
-    <link name="pelvis_link">
+    <link name="torso_link">
       <!-- Visual -->
       <visual>
         <geometry>
-          <box size="0.35 0.30 0.20"/>
+          <box size="0.45 0.30 0.55"/>
         </geometry>
         <origin
           xyz="0 0 0"/>
-        <material name="pelvis_blue"/>
+        <material name="torso_blue"/>
       </visual>
       <!-- Collision -->
       <collision>
         <geometry>
-          <box size="0.35 0.30 0.20"/>
+          <box size="0.45 0.30 0.55"/>
         </geometry>
         <origin
@@ -34,16 +34,26 @@
       <!-- Inertial -->
       <inertial>
-        <mass value="2.5"/>
+        <mass value="5.0"/>
         <origin
           xyz="0 0 0"/>
         <inertia
-          ixx="0.025"
+          ixx="0.12"
           ixy="0"
           ixz="0"
-          iyy="0.020"
+          iyy="0.10"
           iyz="0"
-          izz="0.015"/>
+          izz="0.08"/>
       </inertial>
     </link>
+    <!-- ================= -->
+    <!-- Torso-Pelvis Joint -->
+    <!-- ================= -->
+    <joint name="torso_joint"
+           type="fixed">
+      <parent link="pelvis_link"/>
+      <child link="torso_link"/>
+      <origin
+        xyz="0 0 0.20"/>
+    </joint>
   </xacro:macro>
 </robot>

File: src/humanoid_description/urdf/humanoid.xacro (robot description, xacro)
@@ -1,26 +1,65 @@
 <?xml version="1.0"?>
 <robot xmlns:xacro="http://www.ros.org/wiki/xacro"
-       name="humanoid_v1_9">
+       name="humanoid_v2_5">
   <!-- ================= -->
   <!-- Include Modules -->
   <!-- ================= -->
   <xacro:include
+    filename="$(find humanoid_description)/urdf/modules/pelvis.xacro"/>
+  <xacro:include
+    filename="$(find humanoid_description)/urdf/modules/torso.xacro"/>
+  <xacro:include
     filename="$(find humanoid_description)/urdf/modules/legs.xacro"/>
   <xacro:include
-    filename="$(find humanoid_description)/urdf/modules/pelvis.xacro"/>
-  <xacro:include
-    filename="$(find humanoid_description)/urdf/modules/torso.xacro"/>
-  <xacro:include
     filename="$(find humanoid_description)/urdf/modules/arms.xacro"/>
   <xacro:include
     filename="$(find humanoid_description)/urdf/modules/head.xacro"/>
   <!-- ================= -->
-  <!-- Root Link -->
-  <!-- ================= -->
-  <link name="base_link"/>
-  <!-- ================= -->
-  <!-- Pelvis -->
+  <!-- Base -->
+  <!-- ================= -->
+  <link name="base_link">
+    <visual>
+      <geometry>
+        <box size="0.4 0.3 0.5"/>
+      </geometry>
+      <origin
+        xyz="0 0 0.25"/>
+      <material name="base_blue">
+        <color rgba="0 0 1 1"/>
+      </material>
+    </visual>
+    <collision>
+      <geometry>
+        <box size="0.4 0.3 0.5"/>
+      </geometry>
+      <origin
+        xyz="0 0 0.25"/>
+    </collision>
+    <inertial>
+      <mass value="5"/>
+      <origin
+        xyz="0 0 0.25"/>
+      <inertia
+        ixx="0.1"
+        ixy="0"
+        ixz="0"
+        iyy="0.1"
+        iyz="0"
+        izz="0.08"/>
+    </inertial>
+  </link>
+  <!-- ================= -->
+  <!-- Generate Modules -->
   <!-- ================= -->
   <xacro:pelvis/>
+  <xacro:torso/>
+  <xacro:leg prefix="left"/>
+  <xacro:leg prefix="right"/>
+  <xacro:arm prefix="left"/>
+  <xacro:arm prefix="right"/>
+  <xacro:head/>
+  <!-- ================= -->
+  <!-- Base To Pelvis -->
+  <!-- ================= -->
   <joint name="base_to_pelvis"
          type="fixed">
@@ -31,7 +70,6 @@
   </joint>
   <!-- ================= -->
-  <!-- Torso -->
-  <!-- ================= -->
-  <xacro:torso/>
+  <!-- Pelvis To Torso -->
+  <!-- ================= -->
   <joint name="pelvis_to_torso"
          type="fixed">
@@ -42,8 +80,6 @@
   </joint>
   <!-- ================= -->
-  <!-- Legs -->
-  <!-- ================= -->
-  <xacro:leg prefix="left"/>
-  <xacro:leg prefix="right"/>
+  <!-- Hip Joints -->
+  <!-- ================= -->
   <joint name="left_hip_joint"
          type="revolute">
@@ -73,15 +109,94 @@
   </joint>
   <!-- ================= -->
-  <!-- Arms -->
-  <!-- ================= -->
-  <xacro:arm
-    prefix="left"
-    side="0.25"/>
-  <xacro:arm
-    prefix="right"
-    side="-0.25"/>
-  <!-- ================= -->
-  <!-- Head -->
-  <!-- ================= -->
-  <xacro:head/>
+  <!-- Shoulder -->
+  <!-- ================= -->
+  <joint name="left_shoulder_joint"
+         type="revolute">
+    <parent link="torso_link"/>
+    <child link="left_upper_arm"/>
+    <origin
+      xyz="0 0.25 0.15"/>
+    <axis xyz="1 0 0"/>
+    <limit
+      lower="-1.57"
+      upper="1.57"
+      effort="30"
+      velocity="2"/>
+  </joint>
+  <joint name="right_shoulder_joint"
+         type="revolute">
+    <parent link="torso_link"/>
+    <child link="right_upper_arm"/>
+    <origin
+      xyz="0 -0.25 0.15"/>
+    <axis xyz="1 0 0"/>
+    <limit
+      lower="-1.57"
+      upper="1.57"
+      effort="30"
+      velocity="2"/>
+  </joint>
+  <!-- ================= -->
+  <!-- Elbows -->
+  <!-- ================= -->
+  <joint name="left_elbow_joint"
+         type="revolute">
+    <parent link="left_upper_arm"/>
+    <child link="left_forearm"/>
+    <origin
+      xyz="0 0 -0.30"/>
+    <axis xyz="1 0 0"/>
+    <limit
+      lower="0"
+      upper="2.5"
+      effort="20"
+      velocity="2"/>
+  </joint>
+  <joint name="right_elbow_joint"
+         type="revolute">
+    <parent link="right_upper_arm"/>
+    <child link="right_forearm"/>
+    <origin
+      xyz="0 0 -0.30"/>
+    <axis xyz="1 0 0"/>
+    <limit
+      lower="0"
+      upper="2.5"
+      effort="20"
+      velocity="2"/>
+  </joint>
+  <!-- ================= -->
+  <!-- Wrist -->
+  <!-- ================= -->
+  <joint name="left_wrist_joint"
+         type="fixed">
+    <parent link="left_forearm"/>
+    <child link="left_hand"/>
+    <origin
+      xyz="0 0 -0.28"/>
+  </joint>
+  <joint name="right_wrist_joint"
+         type="fixed">
+    <parent link="right_forearm"/>
+    <child link="right_hand"/>
+    <origin
+      xyz="0 0 -0.28"/>
+  </joint>
+  <!-- ================= -->
+  <!-- Neck -->
+  <!-- ================= -->
+  <joint name="neck_joint"
+         type="fixed">
+    <parent link="torso_link"/>
+    <child link="neck_link"/>
+    <origin
+      xyz="0 0 0.35"/>
+  </joint>
+  <joint name="head_joint"
+         type="fixed">
+    <parent link="neck_link"/>
+    <child link="head_link"/>
+    <origin
+      xyz="0 0 0.15"/>
+  </joint>
 </robot>

File: src/humanoid_description/urdf/modules/arms.xacro (robot description, xacro)
@@ -5,5 +5,5 @@
   <!-- ===================== -->
   <material name="arm_gray">
-    <color rgba="0.65 0.65 0.65 1"/>
+    <color rgba="0.55 0.55 0.55 1"/>
   </material>
   <material name="hand_black">
@@ -14,5 +14,5 @@
   <!-- ===================== -->
   <xacro:macro name="arm"
-               params="prefix side">
+               params="prefix">
     <!-- ================= -->
     <!-- Upper Arm -->
@@ -22,5 +22,5 @@
         <geometry>
           <cylinder
-            radius="0.045"
+            radius="0.06"
             length="0.30"/>
         </geometry>
@@ -32,5 +32,5 @@
         <geometry>
           <cylinder
-            radius="0.045"
+            radius="0.06"
             length="0.30"/>
         </geometry>
@@ -39,14 +39,14 @@
       </collision>
       <inertial>
-        <mass value="0.8"/>
+        <mass value="1.2"/>
         <origin
           xyz="0 0 -0.15"/>
         <inertia
-          ixx="0.006"
+          ixx="0.012"
           ixy="0"
           ixz="0"
-          iyy="0.006"
+          iyy="0.012"
           iyz="0"
-          izz="0.001"/>
+          izz="0.004"/>
       </inertial>
     </link>
@@ -58,9 +58,9 @@
         <geometry>
           <cylinder
-            radius="0.035"
-            length="0.25"/>
+            radius="0.05"
+            length="0.28"/>
         </geometry>
         <origin
-          xyz="0 0 -0.125"/>
+          xyz="0 0 -0.14"/>
         <material name="arm_gray"/>
       </visual>
@@ -68,21 +68,21 @@
         <geometry>
           <cylinder
-            radius="0.035"
-            length="0.25"/>
+            radius="0.05"
+            length="0.28"/>
         </geometry>
         <origin
-          xyz="0 0 -0.125"/>
+          xyz="0 0 -0.14"/>
       </collision>
       <inertial>
-        <mass value="0.5"/>
+        <mass value="0.8"/>
         <origin
-          xyz="0 0 -0.125"/>
+          xyz="0 0 -0.14"/>
         <inertia
-          ixx="0.003"
+          ixx="0.008"
           ixy="0"
           ixz="0"
-          iyy="0.003"
+          iyy="0.008"
           iyz="0"
-          izz="0.0008"/>
+          izz="0.002"/>
       </inertial>
     </link>
@@ -93,72 +93,30 @@
       <visual>
         <geometry>
-          <box size="0.12 0.08 0.05"/>
+          <box size="0.16 0.10 0.08"/>
         </geometry>
         <origin
-          xyz="0 -0.02 -0.025"/>
+          xyz="0 0 -0.04"/>
         <material name="hand_black"/>
       </visual>
       <collision>
         <geometry>
-          <box size="0.12 0.08 0.05"/>
+          <box size="0.16 0.10 0.08"/>
         </geometry>
         <origin
-          xyz="0 -0.02 -0.025"/>
+          xyz="0 0 -0.04"/>
       </collision>
       <inertial>
-        <mass value="0.2"/>
+        <mass value="0.3"/>
         <origin
-          xyz="0 -0.02 -0.025"/>
+          xyz="0 0 -0.04"/>
         <inertia
-          ixx="0.0005"
+          ixx="0.002"
           ixy="0"
           ixz="0"
-          iyy="0.0005"
+          iyy="0.002"
           iyz="0"
-          izz="0.0005"/>
+          izz="0.001"/>
       </inertial>
     </link>
-    <!-- ================= -->
-    <!-- Shoulder Joint -->
-    <!-- ================= -->
-    <joint name="${prefix}_shoulder_joint"
-           type="revolute">
-      <parent link="torso_link"/>
-      <child link="${prefix}_upper_arm"/>
-      <origin
-        xyz="0 ${side} 0.15"/>
-      <axis xyz="1 0 0"/>
-      <limit
-        lower="-1.57"
-        upper="1.57"
-        effort="30"
-        velocity="2"/>
-    </joint>
-    <!-- ================= -->
-    <!-- Elbow Joint -->
-    <!-- ================= -->
-    <joint name="${prefix}_elbow_joint"
-           type="revolute">
-      <parent link="${prefix}_upper_arm"/>
-      <child link="${prefix}_forearm"/>
-      <origin
-        xyz="0 0 -0.30"/>
-      <axis xyz="1 0 0"/>
-      <limit
-        lower="-2.0"
-        upper="0"
-        effort="20"
-        velocity="2"/>
-    </joint>
-    <!-- ================= -->
-    <!-- Wrist Joint -->
-    <!-- ================= -->
-    <joint name="${prefix}_wrist_joint"
-           type="fixed">
-      <parent link="${prefix}_forearm"/>
-      <child link="${prefix}_hand"/>
-      <origin
-        xyz="0 0 -0.25"/>
-    </joint>
   </xacro:macro>
 </robot>
