Commit message: Humanoid Robot v2.8.0: Complete humanoid URDF architecture

File: src/humanoid_description/backup/humanoid_v2.8_before_arm_fix.xacro (robot description, xacro)
@@ -1,5 +1,5 @@
 <?xml version="1.0"?>
 <robot xmlns:xacro="http://www.ros.org/wiki/xacro"
-       name="humanoid_v2_8">
+       name="humanoid_v2_5">
   <!-- ================= -->
   <!-- Include Modules -->
@@ -74,15 +74,11 @@
   <!-- Legs -->
   <!-- ================= -->
-  <xacro:leg prefix="left"
-             side_y="0.15"/>
-  <xacro:leg prefix="right"
-             side_y="0.15"/>
+  <xacro:leg prefix="left"/>
+  <xacro:leg prefix="right"/>
   <!-- ================= -->
   <!-- Arms -->
   <!-- ================= -->
-  <xacro:arm prefix="left"
-             side_y="0.25"/>
-  <xacro:arm prefix="right"
-             side_y="0.25"/>
+  <xacro:arm prefix="left"/>
+  <xacro:arm prefix="right"/>
   <!-- ================= -->
   <!-- Head -->

File: src/humanoid_description/urdf/humanoid_v2.8_failed_backup.xacro (robot description, xacro)
@@ -3,5 +3,5 @@
        name="humanoid_v2_8">
   <!-- ================= -->
-  <!-- Include Modules -->
+  <!-- Modules -->
   <!-- ================= -->
   <xacro:include
@@ -15,4 +15,7 @@
   <xacro:include
     filename="$(find humanoid_description)/urdf/modules/head.xacro"/>
+  <!-- ROS2 Control -->
+  <xacro:include
+    filename="$(find humanoid_description)/urdf/modules/ros2_control.xacro"/>
   <!-- ================= -->
   <!-- Base -->
@@ -23,6 +26,5 @@
         <box size="0.4 0.25 0.5"/>
       </geometry>
-      <origin
-        xyz="0 0 0.25"/>
+      <origin xyz="0 0 0.25"/>
       <material name="blue">
         <color rgba="0 0 1 1"/>
@@ -33,11 +35,9 @@
         <box size="0.4 0.25 0.5"/>
       </geometry>
-      <origin
-        xyz="0 0 0.25"/>
+      <origin xyz="0 0 0.25"/>
     </collision>
     <inertial>
       <mass value="5"/>
-      <origin
-        xyz="0 0 0.25"/>
+      <origin xyz="0 0 0.25"/>
       <inertia
         ixx="0.05"
@@ -57,6 +57,5 @@
     <parent link="base_link"/>
     <child link="pelvis_link"/>
-    <origin
-      xyz="0 0 0.85"/>
+    <origin xyz="0 0 0.85"/>
   </joint>
   <!-- ================= -->
@@ -68,21 +67,16 @@
     <parent link="pelvis_link"/>
     <child link="torso_link"/>
-    <origin
-      xyz="0 0 0.35"/>
+    <origin xyz="0 0 0.35"/>
   </joint>
   <!-- ================= -->
   <!-- Legs -->
   <!-- ================= -->
-  <xacro:leg prefix="left"
-             side_y="0.15"/>
-  <xacro:leg prefix="right"
-             side_y="0.15"/>
+  <xacro:leg prefix="left"/>
+  <xacro:leg prefix="right"/>
   <!-- ================= -->
   <!-- Arms -->
   <!-- ================= -->
-  <xacro:arm prefix="left"
-             side_y="0.25"/>
-  <xacro:arm prefix="right"
-             side_y="0.25"/>
+  <xacro:arm prefix="left"/>
+  <xacro:arm prefix="right"/>
   <!-- ================= -->
   <!-- Head -->

File: src/humanoid_description/urdf/modules/arms_v2.8_broken_backup.xacro (robot description, xacro)
@@ -1,4 +1,7 @@
 <?xml version="1.0"?>
 <robot xmlns:xacro="http://www.ros.org/wiki/xacro">
+  <!-- ===================== -->
+  <!-- Materials -->
+  <!-- ===================== -->
   <material name="arm_gray">
     <color rgba="0.55 0.55 0.55 1"/>
@@ -7,26 +10,36 @@
     <color rgba="0.1 0.1 0.1 1"/>
   </material>
+  <!-- ===================== -->
+  <!-- Arm Macro -->
+  <!-- ===================== -->
   <xacro:macro name="arm"
-               params="prefix side_y">
+               params="prefix">
+    <!-- ================= -->
     <!-- Upper Arm -->
+    <!-- ================= -->
     <link name="${prefix}_upper_arm">
       <visual>
         <geometry>
-          <cylinder radius="0.06"
-                    length="0.30"/>
+          <cylinder
+            radius="0.06"
+            length="0.30"/>
         </geometry>
-        <origin xyz="0 0 -0.15"/>
+        <origin
+          xyz="0 0 -0.15"/>
         <material name="arm_gray"/>
       </visual>
       <collision>
         <geometry>
-          <cylinder radius="0.06"
-                    length="0.30"/>
+          <cylinder
+            radius="0.06"
+            length="0.30"/>
         </geometry>
-        <origin xyz="0 0 -0.15"/>
+        <origin
+          xyz="0 0 -0.15"/>
       </collision>
       <inertial>
         <mass value="1.2"/>
-        <origin xyz="0 0 -0.15"/>
+        <origin
+          xyz="0 0 -0.15"/>
         <inertia
           ixx="0.012"
@@ -38,24 +51,31 @@
       </inertial>
     </link>
+    <!-- ================= -->
     <!-- Forearm -->
+    <!-- ================= -->
     <link name="${prefix}_forearm">
       <visual>
         <geometry>
-          <cylinder radius="0.05"
-                    length="0.28"/>
+          <cylinder
+            radius="0.05"
+            length="0.28"/>
         </geometry>
-        <origin xyz="0 0 -0.14"/>
+        <origin
+          xyz="0 0 -0.14"/>
         <material name="arm_gray"/>
       </visual>
       <collision>
         <geometry>
-          <cylinder radius="0.05"
-                    length="0.28"/>
+          <cylinder
+            radius="0.05"
+            length="0.28"/>
         </geometry>
-        <origin xyz="0 0 -0.14"/>
+        <origin
+          xyz="0 0 -0.14"/>
       </collision>
       <inertial>
         <mass value="0.8"/>
-        <origin xyz="0 0 -0.14"/>
+        <origin
+          xyz="0 0 -0.14"/>
         <inertia
           ixx="0.008"
@@ -67,5 +87,7 @@
       </inertial>
     </link>
+    <!-- ================= -->
     <!-- Hand -->
+    <!-- ================= -->
     <link name="${prefix}_hand">
       <visual>
@@ -73,5 +95,6 @@
           <box size="0.16 0.10 0.08"/>
         </geometry>
-        <origin xyz="0 0 -0.04"/>
+        <origin
+          xyz="0 0 -0.04"/>
         <material name="hand_black"/>
       </visual>
@@ -80,9 +103,11 @@
           <box size="0.16 0.10 0.08"/>
         </geometry>
-        <origin xyz="0 0 -0.04"/>
+        <origin
+          xyz="0 0 -0.04"/>
       </collision>
       <inertial>
         <mass value="0.3"/>
-        <origin xyz="0 0 -0.04"/>
+        <origin
+          xyz="0 0 -0.04"/>
         <inertia
           ixx="0.002"
@@ -94,37 +119,4 @@
       </inertial>
     </link>
-    <!-- Shoulder -->
-    <joint name="${prefix}_shoulder_joint"
-           type="revolute">
-      <parent link="torso_link"/>
-      <child link="${prefix}_upper_arm"/>
-      <origin xyz="0 ${side_y} 0.15"/>
-      <axis xyz="1 0 0"/>
-      <limit
-        effort="30"
-        lower="-1.57"
-        upper="1.57"
-        velocity="2"/>
-    </joint>
-    <!-- Elbow -->
-    <joint name="${prefix}_elbow_joint"
-           type="revolute">
-      <parent link="${prefix}_upper_arm"/>
-      <child link="${prefix}_forearm"/>
-      <origin xyz="0 0 -0.30"/>
-      <axis xyz="1 0 0"/>
-      <limit
-        effort="20"
-        lower="-1.57"
-        upper="1.57"
-        velocity="2"/>
-    </joint>
-    <!-- Wrist -->
-    <joint name="${prefix}_wrist_joint"
-           type="fixed">
-      <parent link="${prefix}_forearm"/>
-      <child link="${prefix}_hand"/>
-      <origin xyz="0 0 -0.28"/>
-    </joint>
   </xacro:macro>
 </robot>

File: src/humanoid_description/urdf/modules/arms_v2.8_failed_variable_backup.xacro (robot description, xacro)
@@ -8,5 +8,5 @@
   </material>
   <xacro:macro name="arm"
-               params="prefix side_y">
+               params="prefix">
     <!-- Upper Arm -->
     <link name="${prefix}_upper_arm">
@@ -94,10 +94,11 @@
       </inertial>
     </link>
-    <!-- Shoulder -->
+    <!-- Shoulder Joint -->
     <joint name="${prefix}_shoulder_joint"
            type="revolute">
       <parent link="torso_link"/>
       <child link="${prefix}_upper_arm"/>
-      <origin xyz="0 ${side_y} 0.15"/>
+      <origin
+        xyz="0 ${prefix}_arm_y 0.15"/>
       <axis xyz="1 0 0"/>
       <limit
@@ -107,10 +108,11 @@
         velocity="2"/>
     </joint>
-    <!-- Elbow -->
+    <!-- Elbow Joint -->
     <joint name="${prefix}_elbow_joint"
            type="revolute">
       <parent link="${prefix}_upper_arm"/>
       <child link="${prefix}_forearm"/>
-      <origin xyz="0 0 -0.30"/>
+      <origin
+        xyz="0 0 -0.30"/>
       <axis xyz="1 0 0"/>
       <limit
@@ -120,10 +122,11 @@
         velocity="2"/>
     </joint>
-    <!-- Wrist -->
+    <!-- Wrist Joint -->
     <joint name="${prefix}_wrist_joint"
            type="fixed">
       <parent link="${prefix}_forearm"/>
       <child link="${prefix}_hand"/>
-      <origin xyz="0 0 -0.28"/>
+      <origin
+        xyz="0 0 -0.28"/>
     </joint>
   </xacro:macro>

File: src/humanoid_description/urdf/modules/head_v2.8_before_fix.xacro (robot description, xacro)
@@ -11,5 +11,6 @@
   </material>
   <!-- ================= -->
-  <!-- Head Macro -->
+  <!-- Head Module -->
+  <!-- V2.8.0 -->
   <!-- ================= -->
   <xacro:macro name="head">
@@ -24,5 +25,6 @@
             length="0.20"/>
         </geometry>
-        <origin xyz="0 0 0"/>
+        <origin
+          xyz="0 0 0"/>
         <material name="neck_dark"/>
       </visual>
@@ -33,9 +35,11 @@
             length="0.20"/>
         </geometry>
-        <origin xyz="0 0 0"/>
+        <origin
+          xyz="0 0 0"/>
       </collision>
       <inertial>
         <mass value="0.5"/>
-        <origin xyz="0 0 0"/>
+        <origin
+          xyz="0 0 0"/>
         <inertia
           ixx="0.002"
@@ -55,5 +59,6 @@
           <sphere radius="0.18"/>
         </geometry>
-        <origin xyz="0 0 0"/>
+        <origin
+          xyz="0 0 0"/>
         <material name="head_gray"/>
       </visual>
@@ -62,9 +67,11 @@
           <sphere radius="0.18"/>
         </geometry>
-        <origin xyz="0 0 0"/>
+        <origin
+          xyz="0 0 0"/>
       </collision>
       <inertial>
         <mass value="1.0"/>
-        <origin xyz="0 0 0"/>
+        <origin
+          xyz="0 0 0"/>
         <inertia
           ixx="0.005"
@@ -77,26 +84,12 @@
     </link>
     <!-- ================= -->
-    <!-- Neck Joint -->
+    <!-- Neck To Head Joint -->
     <!-- ================= -->
     <joint name="neck_joint"
-           type="revolute">
-      <parent link="torso_link"/>
-      <child link="neck_link"/>
-      <origin xyz="0 0 0.35"/>
-      <axis xyz="0 1 0"/>
-      <limit
-        effort="10"
-        lower="-1.0"
-        upper="1.0"
-        velocity="1"/>
-    </joint>
-    <!-- ================= -->
-    <!-- Head Fixed Joint -->
-    <!-- ================= -->
-    <joint name="head_joint"
            type="fixed">
       <parent link="neck_link"/>
       <child link="head_link"/>
-      <origin xyz="0 0 0.20"/>
+      <origin
+        xyz="0 0 0.18"/>
     </joint>
   </xacro:macro>

File: src/humanoid_description/urdf/modules/legs_v2.8_broken_backup.xacro (robot description, xacro)
@@ -1,15 +1,18 @@
 <?xml version="1.0"?>
 <robot xmlns:xacro="http://www.ros.org/wiki/xacro">
-  <!-- ================= -->
+  <!-- ===================== -->
   <!-- Materials -->
-  <!-- ================= -->
+  <!-- ===================== -->
   <material name="leg_gray">
     <color rgba="0.55 0.55 0.55 1"/>
   </material>
-  <!-- ================= -->
-  <!-- Legs Macro -->
-  <!-- ================= -->
+  <material name="foot_black">
+    <color rgba="0.1 0.1 0.1 1"/>
+  </material>
+  <!-- ===================== -->
+  <!-- Leg Macro -->
+  <!-- ===================== -->
   <xacro:macro name="leg"
-               params="prefix side_y">
+               params="prefix">
     <!-- ================= -->
     <!-- Thigh -->
@@ -22,5 +25,6 @@
             length="0.35"/>
         </geometry>
-        <origin xyz="0 0 -0.175"/>
+        <origin
+          xyz="0 0 -0.175"/>
         <material name="leg_gray"/>
       </visual>
@@ -31,9 +35,11 @@
             length="0.35"/>
         </geometry>
-        <origin xyz="0 0 -0.175"/>
+        <origin
+          xyz="0 0 -0.175"/>
       </collision>
       <inertial>
         <mass value="1.5"/>
-        <origin xyz="0 0 -0.175"/>
+        <origin
+          xyz="0 0 -0.175"/>
         <inertia
           ixx="0.015"
@@ -55,5 +61,6 @@
             length="0.35"/>
         </geometry>
-        <origin xyz="0 0 -0.175"/>
+        <origin
+          xyz="0 0 -0.175"/>
         <material name="leg_gray"/>
       </visual>
@@ -64,9 +71,11 @@
             length="0.35"/>
         </geometry>
-        <origin xyz="0 0 -0.175"/>
+        <origin
+          xyz="0 0 -0.175"/>
       </collision>
       <inertial>
         <mass value="1.0"/>
-        <origin xyz="0 0 -0.175"/>
+        <origin
+          xyz="0 0 -0.175"/>
         <inertia
           ixx="0.01"
@@ -84,42 +93,30 @@
       <visual>
         <geometry>
-          <box size="0.25 0.15 0.08"/>
+          <box size="0.25 0.14 0.08"/>
         </geometry>
-        <origin xyz="0 0 -0.04"/>
-        <material name="leg_gray"/>
+        <origin
+          xyz="0.08 0 -0.04"/>
+        <material name="foot_black"/>
       </visual>
       <collision>
         <geometry>
-          <box size="0.25 0.15 0.08"/>
+          <box size="0.25 0.14 0.08"/>
         </geometry>
-        <origin xyz="0 0 -0.04"/>
+        <origin
+          xyz="0.08 0 -0.04"/>
       </collision>
       <inertial>
         <mass value="0.5"/>
-        <origin xyz="0 0 -0.04"/>
+        <origin
+          xyz="0.08 0 -0.04"/>
         <inertia
-          ixx="0.004"
+          ixx="0.002"
           ixy="0"
           ixz="0"
           iyy="0.004"
           iyz="0"
-          izz="0.002"/>
+          izz="0.005"/>
       </inertial>
     </link>
-    <!-- ================= -->
-    <!-- Hip Joint -->
-    <!-- ================= -->
-    <joint name="${prefix}_hip_joint"
-            type="revolute">
-      <parent link="pelvis_link"/>
-      <child link="${prefix}_thigh"/>
-      <origin xyz="0 ${side_y} 0"/>
-      <axis xyz="1 0 0"/>
-      <limit
-        effort="40"
-        lower="-1.57"
-        upper="1.57"
-        velocity="2"/>
-    </joint>
     <!-- ================= -->
     <!-- Knee Joint -->
@@ -129,14 +126,15 @@
       <parent link="${prefix}_thigh"/>
       <child link="${prefix}_shin"/>
-      <origin xyz="0 0 -0.35"/>
+      <origin
+        xyz="0 0 -0.35"/>
       <axis xyz="1 0 0"/>
       <limit
-        effort="30"
-        lower="-1.57"
-        upper="0"
+        lower="0"
+        upper="2.5"
+        effort="50"
         velocity="2"/>
     </joint>
     <!-- ================= -->
-    <!-- Ankle -->
+    <!-- Ankle Joint -->
     <!-- ================= -->
     <joint name="${prefix}_ankle_joint"
@@ -144,5 +142,6 @@
       <parent link="${prefix}_shin"/>
       <child link="${prefix}_foot"/>
-      <origin xyz="0 0 -0.35"/>
+      <origin
+        xyz="0 0 -0.35"/>
     </joint>
   </xacro:macro>
